File: board/assistant.brd (EAGLE design)
At the start: 160 x 105.1 mm, 45 parts, among them IC1 7805T, J1 DCJ0202, K1 RELAY(10A), K2 RELAY(10A), K3 RELAY(10A), T1 TR-2N2222_1, T2 TR-2N2222_1, T3 TR-2N2222_1

Commit message: final board
Connections:
- removed net N$10: D5.C, D6.A, J1.1
- net N$7: now also D5.C, D6.A
- net N$9: now also J1.1
Routing:
- net N$9: track 58.2 -> 108.3 mm
- net N$7: track 30.2 -> 74.8 mm
- net N$10: track 39.5 -> 0.00 mm
Changed lines of the file:
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@@
 <setting verticaltext="up"/>
 </settings>
-<grid distance="0.003125" unitdist="mic" unit="mm" style="lines" multiple="1" display="yes" altdistance="5" altunitdist="mil" altunit="mm"/>
+<grid distance="1.27" unitdist="mm" unit="mm" style="lines" multiple="1" display="yes" altdistance="5" altunitdist="mil" altunit="mm"/>
 <layers>
 <layer number="1" name="Top" color="4" fill="1" visible="yes" active="yes"/>
@@
 </layers>
 <board>
+<fusionsync huburn="a.YnVzaW5lc3M6YWxleHUxMzU" projecturn="a.YnVzaW5lc3M6YWxleHUxMzUjRDIwMjEwOTE5NDQ2MTcyOTgx" f3durn="urn:adsk.wipprod:dm.lineage:hK4Y5Z7YTSGo1YRWdHuAYA" pcbguid="2d551ee5-e54d-4eeb-8952-a6af44ef71ec" lastpulledtime="" lastsyncedchangeguid="" latestrevisionid="7c1c1745-8081-44fc-acf9-ad925d2d41f8" lastsyncedrevisionid="7c1c1745-8081-44fc-acf9-ad925d2d41f8" lastboardhashguid="d1c52d2d-73eb-a542-cd83-84718ada4fd7" lastpushedtime="2023-10-25T00:52:05Z" linktopcb3d="true"/>
 <plain>
 <wire x1="0" y1="0" x2="160" y2="0" width="0" layer="20"/>
@@
 <vertex x="158.75" y="99.06"/>
 </polygon>
+<polygon width="0.8" layer="16" pour="cutout">
+<vertex x="0" y="36.83"/>
+<vertex x="30.48" y="36.83"/>
+<vertex x="30.48" y="1.27"/>
+<vertex x="0" y="1.27"/>
+</polygon>
+<polygon width="0.8" layer="16" pour="cutout">
+<vertex x="30.48" y="12.7"/>
+<vertex x="54.61" y="12.7"/>
+<vertex x="57.15" y="15.24"/>
+<vertex x="60.96" y="15.24"/>
+<vertex x="60.96" y="16.51"/>
+<vertex x="71.12" y="16.51"/>
+<vertex x="71.12" y="0"/>
+<vertex x="30.48" y="0"/>
+</polygon>
+<polygon width="0.8" layer="16" pour="cutout">
+<vertex x="71.12" y="13.97"/>
+<vertex x="78.74" y="13.97"/>
+<vertex x="80.01" y="12.7"/>
+<vertex x="80.01" y="1.27"/>
+<vertex x="71.12" y="1.27"/>
+</polygon>
+<polygon width="0.8" layer="16" pour="cutout">
+<vertex x="81.28" y="15.24"/>
+<vertex x="81.28" y="1.27"/>
+<vertex x="80.01" y="1.27"/>
+<vertex x="78.74" y="2.54"/>
+<vertex x="78.74" y="13.97"/>
+<vertex x="80.01" y="15.24"/>
+</polygon>
+<polygon width="0.8" layer="16" pour="cutout">
+<vertex x="5.58615625" y="90.17"/>
+<vertex x="5.58615625" y="82.55"/>
+<vertex x="7.62" y="82.55"/>
+<vertex x="7.62" y="90.17"/>
+</polygon>
+<polygon width="0.8" layer="16" pour="cutout">
+<vertex x="71.12" y="76.2"/>
+<vertex x="71.12" y="73.66"/>
+<vertex x="72.39" y="72.39"/>
+<vertex x="73.66" y="73.66"/>
+<vertex x="73.66" y="76.2"/>
+</polygon>
+<polygon width="0.8" layer="16" pour="cutout">
+<vertex x="71.12" y="90.17"/>
+<vertex x="73.66" y="90.17"/>
+<vertex x="73.66" y="83.82"/>
+<vertex x="71.12" y="83.82"/>
+</polygon>
+<polygon width="0.8" layer="16" pour="cutout">
+<vertex x="73.66" y="90.17"/>
+<vertex x="78.74" y="90.17"/>
+<vertex x="78.74" y="93.98"/>
+<vertex x="77.47" y="93.98"/>
+</polygon>
+<polygon width="0.8" layer="16" pour="cutout">
+<vertex x="78.74" y="82.55"/>
+<vertex x="73.66" y="82.55"/>
+<vertex x="73.66" y="80.01"/>
+<vertex x="74.93" y="81.28"/>
+<vertex x="78.74" y="81.28"/>
+</polygon>
+<polygon width="0.8" layer="16" pour="cutout">
+<vertex x="73.66" y="55.88"/>
+<vertex x="73.66" y="59.69"/>
+<vertex x="71.12" y="59.69"/>
+<vertex x="71.12" y="55.88"/>
+</polygon>
+<polygon width="0.8" layer="16" pour="cutout">
+<vertex x="88.9" y="26.67"/>
+<vertex x="88.9" y="25.4"/>
+<vertex x="87.63" y="24.13"/>
+<vertex x="85.09" y="24.13"/>
+<vertex x="83.82" y="25.4"/>
+<vertex x="83.82" y="26.67"/>
+</polygon>
 </signal>
 <signal name="IO15">
@@
 <wire x1="12.7" y1="24.41" x2="9.7" y2="27.41" width="0.8128" layer="16"/>
 <wire x1="9.7" y1="27.41" x2="9.7" y2="29.21" width="0.8128" layer="16"/>
+<contactref element="D6" pad="A"/>
+<contactref element="D5" pad="C"/>
+<wire x1="45.72" y1="19.05" x2="45.72" y2="22.86" width="0.8128" layer="16"/>
+<wire x1="45.72" y1="22.86" x2="39.37" y2="29.21" width="0.8128" layer="16"/>
+<wire x1="39.37" y1="29.21" x2="35.56" y2="33.02" width="0.8128" layer="16"/>
+<wire x1="26.67" y1="33.02" x2="22.86" y2="29.21" width="0.8128" layer="16"/>
+<wire x1="35.56" y1="33.02" x2="26.67" y2="33.02" width="0.8128" layer="16"/>
+<wire x1="22.86" y1="29.21" x2="18.06" y2="24.41" width="0.8" layer="16"/>
+<wire x1="18.06" y1="24.41" x2="12.7" y2="24.41" width="0.8" layer="16"/>
 </signal>
 <signal name="N$9">
@@
 <wire x1="26.67" y1="25.4" x2="30.48" y2="29.21" width="0.8128" layer="16"/>
 <wire x1="30.48" y1="29.21" x2="31.75" y2="29.21" width="0.8128" layer="16"/>
-</signal>
-<signal name="N$10">
 <contactref element="J1" pad="1"/>
-<contactref element="D6" pad="A"/>
-<contactref element="D5" pad="C"/>
-<wire x1="45.72" y1="19.05" x2="45.72" y2="22.86" width="0.8128" layer="16"/>
-<wire x1="45.72" y1="22.86" x2="39.37" y2="29.21" width="0.8128" layer="16"/>
-<wire x1="39.37" y1="29.21" x2="35.56" y2="33.02" width="0.8128" layer="16"/>
-<wire x1="26.67" y1="33.02" x2="22.86" y2="29.21" width="0.8128" layer="16"/>
-<wire x1="22.86" y1="29.21" x2="15.8" y2="29.21" width="0.8128" layer="16"/>
-<wire x1="35.56" y1="33.02" x2="26.67" y2="33.02" width="0.8128" layer="16"/>
+<wire x1="15.8" y1="29.21" x2="15.8" y2="33.903365625" width="0.8" layer="16"/>
+<wire x1="15.8" y1="33.903365625" x2="14.49701875" y2="35.206346875" width="0.8" layer="16"/>
+<wire x1="14.49701875" y1="35.206346875" x2="7.383459375" y2="35.206346875" width="0.8" layer="16"/>
+<wire x1="7.383459375" y1="35.206346875" x2="6.71158125" y2="34.53446875" width="0.8" layer="16"/>
+<wire x1="6.71158125" y1="34.53446875" x2="3.490021875" y2="31.312909375" width="0.8" layer="16"/>
+<wire x1="3.490021875" y1="31.312909375" x2="3.490021875" y2="10.481278125" width="0.8" layer="16"/>
+<wire x1="3.490021875" y1="10.481278125" x2="3.490021875" y2="9.265146875" width="0.8" layer="16"/>
+<wire x1="3.490021875" y1="9.265146875" x2="9.798909375" y2="2.956259375" width="0.8" layer="16"/>
+<wire x1="15.8" y1="29.21" x2="16.43" y2="16.43" width="0" layer="19" extent="1-1"/>
 </signal>
 <signal name="N$13">
@@
 </note>
 <note version="8.3" severity="warning">
+Since Version 8.3, EAGLE supports Fusion synchronisation.
+This feature will not be available in this version and saving
+the document will break the link to the Fusion PCB feature.
+</note>
+<note version="8.3" severity="warning">
